Commit message: clean&reset the repositories

File: simulation_ws/src/racecar_description/urdf/racecar.urdf (robot description, URDF)
Before this commit: robot origins, 8 links, 7 joints
Links:
- removed link ground_link
- removed link left_front_steering_wheel_link
- removed link right_front_steering_wheel_link
- added link base_footprint
- added link left_front_steering_link, mass 0.5
- added link lidar_link, mass 1.0; collision cylinder length=0.10 radius=0.08; visual cylinder length=0.10 radius=0.08
- added link right_front_steering_link, mass 0.5
- link base_link: mass None -> 180.0; geometry collision box size=2.60 0.75 0.30; visual mesh filename=package://racecar_description/urdf/chassis_lowpoly.stl scale=1 1 1
- link left_front_wheel_link: mass None -> 4.0; geometry collision cylinder length=0.18 radius=0.225; visual mesh filename=package://racecar_description/urdf/left_wheel_lowpoly.stl scale=1 1 1
- link left_rear_wheel_link: mass None -> 4.0; geometry collision cylinder length=0.18 radius=0.225; visual mesh filename=package://racecar_description/urdf/left_wheel_lowpoly.stl scale=1 1 1
- link right_front_wheel_link: mass None -> 4.0; geometry collision cylinder length=0.18 radius=0.225; visual mesh filename=package://racecar_description/urdf/right_wheel_lowpoly.stl scale=1 1 1
- link right_rear_wheel_link: mass None -> 4.0; geometry collision cylinder length=0.18 radius=0.225; visual mesh filename=package://racecar_description/urdf/right_wheel_lowpoly.stl scale=1 1 1
Joints:
- removed joint ground_link
- removed joint left_front_steering_wheel_link
- removed joint left_front_wheel_link
- removed joint left_rear_wheel_link
- removed joint right_front_steering_wheel_link
- removed joint right_front_wheel_link
- removed joint right_rear_wheel_link
- added joint base_footprint_joint: type fixed, parent base_footprint, child base_link
- added joint left_front_steering_joint: type revolute, parent base_link, child left_front_steering_link, origin xyz=1.6 0.59 0, axis 0 0 1, limit lower=-0.52359 upper=0.52359 effort=500 velocity=3.0
- added joint left_front_wheel_joint: type continuous, parent left_front_steering_link, child left_front_wheel_link, axis 0 1 0
- added joint left_rear_wheel_joint: type continuous, parent base_link, child left_rear_wheel_link, origin xyz=0 0.59 0, axis 0 1 0
- added joint lidar_fixed_joint: type fixed, parent base_link, child lidar_link, origin xyz=0.95 0 0.73 rpy=0 0 0
- added joint right_front_steering_joint: type revolute, parent base_link, child right_front_steering_link, origin xyz=1.6 -0.59 0, axis 0 0 1, limit lower=-0.52359 upper=0.52359 effort=500 velocity=3.0
- added joint right_front_wheel_joint: type continuous, parent right_front_steering_link, child right_front_wheel_link, axis 0 1 0
- added joint right_rear_wheel_joint: type continuous, parent base_link, child right_rear_wheel_link, origin xyz=0 -0.59 0, axis 0 1 0

Commit message: optimize launch.py layout

File: simulation_ws/src/racecar_description/urdf/racecar.urdf (robot description, URDF)
Before this commit: robot racecar, 9 links, 8 joints
Joints:
- joint base_footprint_joint: origin (none) -> xyz=0 0 0.225 rpy=0 0 0
- joint lidar_fixed_joint: origin xyz=0.95 0 0.73 rpy=0 0 0 -> xyz=0.95 0 0.955 rpy=0 0 0
